File: PCB/USBC.kicad_sch (KiCad schematic)
At the start: 4 parts, among them J1 USB_C_Receptacle_USB2.0

Commit message: jlcpcb production fixes
Parts:
- D1: JLCPCB Rotation Offset (none) -> 90
- J1: JLCPCB Position Offset (none) -> 0,1.42
Changed lines of the file:
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@@
+			)
+		)
+		(property "JLCPCB Position Offset" "0,1.42"
+			(at 27.94 46.99 0)
+			(effects
+				(font
+					(size 1.27 1.27)
+				)
+				(hide yes)
 			)
 		)
@@
 			(at 95.25 54.61 0)
 			(effects
+				(font
+					(size 1.27 1.27)
+				)
+				(hide yes)
+			)
+		)
+		(property "JLCPCB Rotation Offset" "90"
+			(at 95.25 54.61 0)
+			(effects
